File: mechanic.kicad_sch (KiCad schematic)
At the start: 20 parts

Commit message: 暂存: 基本完成原理图(差雷达接口)
Parts:
- H1, H2, H3, H4: footprint (none) -> MountingHole:MountingHole_2.5mm_Pad_Via
- H10: renamed from H18; footprint (none) -> MountingHole:MountingHole_3.2mm_M3_Pad_Via
- H11: renamed from H9; footprint (none) -> MountingHole:MountingHole_2.5mm_Pad_Via
- H12: renamed from H10; footprint (none) -> MountingHole:MountingHole_2.5mm_Pad_Via
- H13: renamed from H11; footprint (none) -> MountingHole:MountingHole_2.5mm_Pad_Via
- H14: renamed from H12; footprint (none) -> MountingHole:MountingHole_2.5mm_Pad_Via
- H15: renamed from H19; footprint (none) -> MountingHole:MountingHole_3.2mm_M3_Pad_Via
- H16: renamed from H13; footprint (none) -> MountingHole:MountingHole_2.5mm_Pad_Via
- H17: renamed from H14; footprint (none) -> MountingHole:MountingHole_2.5mm_Pad_Via
- H18: renamed from H15; footprint (none) -> MountingHole:MountingHole_2.5mm_Pad_Via
- H19: renamed from H16; footprint (none) -> MountingHole:MountingHole_2.5mm_Pad_Via
- H20: footprint (none) -> MountingHole:MountingHole_3.2mm_M3_Pad_Via
- H5: renamed from H17; footprint (none) -> MountingHole:MountingHole_3.2mm_M3_Pad_Via
- H6: renamed from H5; footprint (none) -> MountingHole:MountingHole_2.5mm_Pad_Via
- H7: renamed from H6; footprint (none) -> MountingHole:MountingHole_2.5mm_Pad_Via
- H8: renamed from H7; footprint (none) -> MountingHole:MountingHole_2.5mm_Pad_Via
- H9: renamed from H8; footprint (none) -> MountingHole:MountingHole_2.5mm_Pad_Via
Changed lines of the file:
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@@
 		(dnp no)
 		(fields_autoplaced yes)
-		(property "Reference" "H10"
+		(property "Reference" "H12"
 			(at 102.87 40.6399 0)
 			(effects
@@
 			)
 		)
-		(property "Footprint" ""
+		(property "Footprint" "MountingHole:MountingHole_2.5mm_Pad_Via"
 			(at 100.33 43.18 0)
 			(effects
@@
 			(project "ZW1S"
 				(path "/c658c753-a869-4eb9-a520-6b2e7fae7fd9/61ba284f-105d-4546-8722-74f9b4410c5d"
-					(reference "H10")
+					(reference "H12")
 					(unit 1)
 				)
@@
 		(dnp no)
 		(fields_autoplaced yes)
-		(property "Reference" "H15"
+		(property "Reference" "H18"
 			(at 135.89 48.2599 0)
 			(effects
@@
 			)
 		)
-		(property "Footprint" ""
+		(property "Footprint" "MountingHole:MountingHole_2.5mm_Pad_Via"
 			(at 133.35 50.8 0)
 			(effects
@@
 			(project "ZW1S"
 				(path "/c658c753-a869-4eb9-a520-6b2e7fae7fd9/61ba284f-105d-4546-8722-74f9b4410c5d"
-					(reference "H15")
+					(reference "H18")
 					(unit 1)
 				)
@@
 		(dnp no)
 		(fields_autoplaced yes)
-		(property "Reference" "H16"
+		(property "Reference" "H19"
 			(at 135.89 55.8799 0)
 			(effects
@@
 			)
 		)
-		(property "Footprint" ""
+		(property "Footprint" "MountingHole:MountingHole_2.5mm_Pad_Via"
 			(at 133.35 58.42 0)
 			(effects
@@
 			(project "ZW1S"
 				(path "/c658c753-a869-4eb9-a520-6b2e7fae7fd9/61ba284f-105d-4546-8722-74f9b4410c5d"
-					(reference "H16")
+					(reference "H19")
 					(unit 1)
 				)
@@
 		(dnp no)
 		(fields_autoplaced yes)
-		(property "Reference" "H9"
+		(property "Reference" "H11"
 			(at 102.87 33.0199 0)
 			(effects
@@
 			)
 		)
-		(property "Footprint" ""
+		(property "Footprint" "MountingHole:MountingHole_2.5mm_Pad_Via"
 			(at 100.33 35.56 0)
 			(effects
@@
 			(project "ZW1S"
 				(path "/c658c753-a869-4eb9-a520-6b2e7fae7fd9/61ba284f-105d-4546-8722-74f9b4410c5d"
-					(reference "H9")
+					(reference "H11")
 					(unit 1)
 				)
@@
 			)
 		)
-		(property "Footprint" ""
+		(property "Footprint" "MountingHole:MountingHole_2.5mm_Pad_Via"
 			(at 34.29 35.56 0)
 			(effects
@@
 		(dnp no)
 		(fields_autoplaced yes)
-		(property "Reference" "H6"
+		(property "Reference" "H7"
 			(at 69.85 40.6399 0)
 			(effects
@@
 			)
 		)
-		(property "Footprint" ""
+		(property "Footprint" "MountingHole:MountingHole_2.5mm_Pad_Via"
 			(at 67.31 43.18 0)
 			(effects
@@
 			(project "ZW1S"
 				(path "/c658c753-a869-4eb9-a520-6b2e7fae7fd9/61ba284f-105d-4546-8722-74f9b4410c5d"
-					(reference "H6")
+					(reference "H7")
 					(unit 1)
 				)
@@
 			)
 		)
-		(property "Footprint" ""
+		(property "Footprint" "MountingHole:MountingHole_2.5mm_Pad_Via"
 			(at 34.29 43.18 0)
 			(effects
@@
 		(dnp no)
 		(fields_autoplaced yes)
-		(property "Reference" "H13"
+		(property "Reference" "H16"
 			(at 135.89 33.0199 0)
 			(effects
@@
 			)
 		)
-		(property "Footprint" ""
+		(property "Footprint" "MountingHole:MountingHole_2.5mm_Pad_Via"
 			(at 133.35 35.56 0)
 			(effects
@@
 			(project "ZW1S"
 				(path "/c658c753-a869-4eb9-a520-6b2e7fae7fd9/61ba284f-105d-4546-8722-74f9b4410c5d"
-					(reference "H13")
+					(reference "H16")
 					(unit 1)
 				)
@@
 		(dnp no)
 		(fields_autoplaced yes)
-		(property "Reference" "H14"
+		(property "Reference" "H17"
 			(at 135.89 40.6399 0)
 			(effects
@@
 			)
 		)
-		(property "Footprint" ""
+		(property "Footprint" "MountingHole:MountingHole_2.5mm_Pad_Via"
 			(at 133.35 43.18 0)
 			(effects
@@
 			(project "ZW1S"
 				(path "/c658c753-a869-4eb9-a520-6b2e7fae7fd9/61ba284f-105d-4546-8722-74f9b4410c5d"
-					(reference "H14")
+					(reference "H17")
 					(unit 1)
 				)
@@
 		(dnp no)
 		(fields_autoplaced yes)
-		(property "Reference" "H17"
+		(property "Reference" "H5"
 			(at 36.83 69.8499 0)
 			(effects
@@
 			)
 		)
-		(property "Footprint" ""
+		(property "Footprint" "MountingHole:MountingHole_3.2mm_M3_Pad_Via"
 			(at 34.29 72.39 0)
 			(effects
@@
 			(project "ZW1S"
 				(path "/c658c753-a869-4eb9-a520-6b2e7fae7fd9/61ba284f-105d-4546-8722-74f9b4410c5d"
-					(reference "H17")
+					(reference "H5")
 					(unit 1)
 				)
@@
 		(dnp no)
 		(fields_autoplaced yes)
-		(property "Reference" "H11"
+		(property "Reference" "H13"
 			(at 102.87 48.2599 0)
 			(effects
@@
 			)
 		)
-		(property "Footprint" ""
+		(property "Footprint" "MountingHole:MountingHole_2.5mm_Pad_Via"
 			(at 100.33 50.8 0)
 			(effects
@@
 			(project "ZW1S"
 				(path "/c658c753-a869-4eb9-a520-6b2e7fae7fd9/61ba284f-105d-4546-8722-74f9b4410c5d"
-					(reference "H11")
+					(reference "H13")
 					(unit 1)
 				)
@@
 		(dnp no)
 		(fields_autoplaced yes)
-		(property "Reference" "H7"
+		(property "Reference" "H8"
 			(at 69.85 48.2599 0)
 			(effects
@@
 			)
 		)
-		(property "Footprint" ""
+		(property "Footprint" "MountingHole:MountingHole_2.5mm_Pad_Via"
 			(at 67.31 50.8 0)
 			(effects
@@
 			(project "ZW1S"
 				(path "/c658c753-a869-4eb9-a520-6b2e7fae7fd9/61ba284f-105d-4546-8722-74f9b4410c5d"
-					(reference "H7")
+					(reference "H8")
 					(unit 1)
 				)
@@
 			)
 		)
-		(property "Footprint" ""
+		(property "Footprint" "MountingHole:MountingHole_3.2mm_M3_Pad_Via"
 			(at 133.35 72.39 0)
 			(effects
@@
 			)
 		)
-		(property "Footprint" ""
+		(property "Footprint" "MountingHole:MountingHole_2.5mm_Pad_Via"
 			(at 34.29 50.8 0)
 			(effects
@@
 		(dnp no)
 		(fields_autoplaced yes)
-		(property "Reference" "H18"
+		(property "Reference" "H10"
 			(at 69.85 69.8499 0)
 			(effects
@@
 			)
 		)
-		(property "Footprint" ""
+		(property "Footprint" "MountingHole:MountingHole_3.2mm_M3_Pad_Via"
 			(at 67.31 72.39 0)
 			(effects
@@
 			(project "ZW1S"
 				(path "/c658c753-a869-4eb9-a520-6b2e7fae7fd9/61ba284f-105d-4546-8722-74f9b4410c5d"
-					(reference "H18")
+					(reference "H10")
 					(unit 1)
 				)
@@
 			)
 		)
-		(property "Footprint" ""
+		(property "Footprint" "MountingHole:MountingHole_2.5mm_Pad_Via"
 			(at 34.29 58.42 0)
 			(effects
@@
 		(dnp no)
 		(fields_autoplaced yes)
-		(property "Reference" "H5"
+		(property "Reference" "H6"
 			(at 69.85 33.0199 0)
 			(effects
@@
 			)
 		)
-		(property "Footprint" ""
+		(property "Footprint" "MountingHole:MountingHole_2.5mm_Pad_Via"
 			(at 67.31 35.56 0)
 			(effects
@@
 			(project "ZW1S"
 				(path "/c658c753-a869-4eb9-a520-6b2e7fae7fd9/61ba284f-105d-4546-8722-74f9b4410c5d"
-					(reference "H5")
+					(reference "H6")
 					(unit 1)
 				)
@@
 		(dnp no)
 		(fields_autoplaced yes)
-		(property "Reference" "H19"
+		(property "Reference" "H15"
 			(at 102.87 69.8499 0)
 			(effects
@@
 			)
 		)
-		(property "Footprint" ""
+		(property "Footprint" "MountingHole:MountingHole_3.2mm_M3_Pad_Via"
 			(at 100.33 72.39 0)
 			(effects
@@
 			(project "ZW1S"
 				(path "/c658c753-a869-4eb9-a520-6b2e7fae7fd9/61ba284f-105d-4546-8722-74f9b4410c5d"
-					(reference "H19")
+					(reference "H15")
 					(unit 1)
 				)
@@
 		(dnp no)
 		(fields_autoplaced yes)
-		(property "Reference" "H8"
+		(property "Reference" "H9"
 			(at 69.85 55.8799 0)
 			(effects
@@
 			)
 		)
-		(property "Footprint" ""
+		(property "Footprint" "MountingHole:MountingHole_2.5mm_Pad_Via"
 			(at 67.31 58.42 0)
 			(effects
@@
 			(project "ZW1S"
 				(path "/c658c753-a869-4eb9-a520-6b2e7fae7fd9/61ba284f-105d-4546-8722-74f9b4410c5d"
-					(reference "H8")
+					(reference "H9")
 					(unit 1)
 				)
@@
 		(dnp no)
 		(fields_autoplaced yes)
-		(property "Reference" "H12"
+		(property "Reference" "H14"
 			(at 102.87 55.8799 0)
 			(effects
@@
 			)
 		)
-		(property "Footprint" ""
+		(property "Footprint" "MountingHole:MountingHole_2.5mm_Pad_Via"
 			(at 100.33 58.42 0)
 			(effects
@@
 			(project "ZW1S"
 				(path "/c658c753-a869-4eb9-a520-6b2e7fae7fd9/61ba284f-105d-4546-8722-74f9b4410c5d"
-					(reference "H12")
-					(unit 1)
-				)
+					(reference "H14")
+					(unit 1)
+				)
